Commit message: readme formatting and ws issue fixes

File: reccobot_description/urdf/reccobot_description.urdf (robot description, URDF)
Before this commit: robot reccobot_description, 44 links, 43 joints
Links:
- added link world
Joints:
- added joint world_to_base: type fixed, parent world, child base_link, origin xyz=0 0 0 rpy=0 0 1.5708

Commit message: origin and mass origin fix

File: reccobot_description/urdf/reccobot_description.urdf (robot description, URDF)
Before this commit: robot reccobot_description, 45 links, 44 joints
Joints:
- joint world_to_base: origin xyz=0 0 0 rpy=0 0 1.5708 -> xyz=0 0 0 rpy=-1.5708 0 0

Commit message: mass update

File: reccobot_description/urdf/reccobot_description.urdf (robot description, URDF)
Before this commit: robot reccobot_description, 45 links, 44 joints
Links:
- link base_link: mass 0.216733439424429 -> 0.21673
