Commit message: controller gazebo fix multiple spwan is still pending

File: reccobot_description/urdf/lidar.xacro (robot description, xacro)
@@ -54,5 +54,5 @@
                 </noise>
             </ray>
-            <plugin name="laser_controller" filename="libgazebo_ros_ray_sensor.so">
+            <plugin name="laser_controller" filename="libgz_ros_lidar_sensor.so">
                 <ros>
                     <argument>~/out:=scan</argument>

File: reccobot_description/urdf/reccobot_description.urdf (robot description, URDF)
Before this commit: robot reccobot_description, 44 links, 43 joints
Links:
- removed link world
- added link chassis_link, mass 0.21673; collision mesh filename=package://reccobot_description/meshes/base_link.STL; visual mesh filename=package://reccobot_description/meshes/base_link.STL
- link base_link: mass 0.21673 -> None; geometry 
Joints:
- removed joint world_to_base
- added joint base_to_chassis: type fixed, parent base_link, child chassis_link, origin xyz=0.0 0.0 0.15 rpy=-1.5708 0 0
- joint base_cambase: limit lower=-1.396 upper=1.396 effort=0.8 velocity=5.0 -> (none); parent base_link -> chassis_link
- joint base_cell1: parent base_link -> chassis_link
- joint base_cell2: parent base_link -> chassis_link
- joint base_cell3: parent base_link -> chassis_link
- joint base_encoder: parent base_link -> chassis_link
- joint base_lipo: parent base_link -> chassis_link
- joint base_servo11: parent base_link -> chassis_link
- joint base_servo21: parent base_link -> chassis_link
- joint base_servo31: parent base_link -> chassis_link
- joint base_servo41: parent base_link -> chassis_link
- joint base_stepper: parent base_link -> chassis_link
- joint camj: limit lower=-1.396 upper=1.396 effort=0.8 velocity=5.0 -> (none)
- joint coxa1_servo12: limit lower=-1.396 upper=1.396 effort=1.2 velocity=6.0 -> (none)
- joint coxa2l_servo2l: limit lower=-1.396 upper=1.396 effort=1.2 velocity=6.0 -> (none)
- joint coxa3l_servo32: limit lower=-1.396 upper=1.396 effort=1.2 velocity=6.0 -> (none)
- joint coxa4l_servo42: limit lower=-1.396 upper=1.396 effort=1.2 velocity=6.0 -> (none)
- joint flange_lidarmount: limit lower=-6.283 upper=6.283 effort=2.5 velocity=3.5 -> (none)
- joint imuj: parent base_link -> chassis_link
- joint servo13_tibia1l: limit lower=-1.396 upper=1.396 effort=1.2 velocity=6.0 -> (none)
- joint servo23_tibia2j: limit lower=-1.396 upper=1.396 effort=1.2 velocity=6.0 -> (none)
- joint servo33_tibia3l: limit lower=-1.396 upper=1.396 effort=1.2 velocity=6.0 -> (none)
- joint servo43_tibia4l: limit lower=-1.396 upper=1.396 effort=1.2 velocity=6.0 -> (none)

File: reccobot_description/urdf/reccobot_gazebo.xacro (robot description, xacro)
@@ -1,3 +1,6 @@
-<!-- Gazebo tuning snippet for reccobot: insert into your URDF under <robot> -->
+<?xml version="1.0"?>
+<!-- Gazebo tuning snippet for reccobot -->
+<!-- Note: ros2_control plugin is defined in reccobot_ros2_control.xacro -->
+<robot xmlns:xacro="http://www.ros.org/wiki/xacro">
 <gazebo reference="coxa1j">
   <kp>80</kp>
@@ -27,5 +30,5 @@
   <provideFeedback>true</provideFeedback>
 </gazebo>
-<gazebo reference="foot1j">
+<gazebo reference="feet1j">
   <kp>80</kp>
   <ki>0.5</ki>
@@ -63,5 +66,5 @@
   <provideFeedback>true</provideFeedback>
 </gazebo>
-<gazebo reference="foot2j">
+<gazebo reference="feet2j">
   <kp>80</kp>
   <ki>0.5</ki>
@@ -99,5 +102,5 @@
   <provideFeedback>true</provideFeedback>
 </gazebo>
-<gazebo reference="foot3j">
+<gazebo reference="feet3j">
   <kp>80</kp>
   <ki>0.5</ki>
@@ -135,5 +138,5 @@
   <provideFeedback>true</provideFeedback>
 </gazebo>
-<gazebo reference="foot4j">
+<gazebo reference="feet4j">
   <kp>80</kp>
   <ki>0.5</ki>
@@ -153,5 +156,6 @@
   <provideFeedback>true</provideFeedback>
 </gazebo>
-<gazebo reference="lidar1j">
+<!-- Lidar rotation joint (base_coupling) -->
+<gazebo reference="base_coupling">
   <kp>5</kp>
   <ki>0.0</ki>
@@ -159,5 +163,6 @@
   <friction>0.01</friction>
   <damping>0.02</damping>
-  <maxEffort>0.255</maxEffort>
+  <maxEffort>0.5</maxEffort>
   <provideFeedback>true</provideFeedback>
 </gazebo>
+</robot>

File: reccobot_description/urdf/reccobot_ros2_control.xacro (robot description, xacro)
@@ -1,4 +1,5 @@
 <?xml version="1.0"?>
 <robot xmlns:xacro="http://www.ros.org/wiki/xacro" name="reccobot">
+  <!-- Ignition/GZ plugin used unconditionally (launch uses ros_gz_sim) -->
   <xacro:property name="PI" value="3.14159265359" />
   <xacro:property name="limit_servo" value="1.396" />
@@ -109,6 +110,14 @@
       <state_interface name="position"/>
     </joint>
+    <!-- Lidar rotation joint -->
+    <joint name="base_coupling">
+      <command_interface name="position">
+        <param name="min">-6.28</param>
+        <param name="max">6.28</param>
+      </command_interface>
+      <state_interface name="position"/>
+    </joint>
   </ros2_control>
-  <!-- Ignition Gazebo ROS 2 Control plugin (Fortress/Garden via ros_gz_sim) -->
+  <!-- ros2_control plugin injection for Ignition Gazebo (ros_gz_sim) -->
   <gazebo>
     <plugin name="ign_ros2_control::IgnitionROS2ControlPlugin" filename="libign_ros2_control-system.so">
