Commit message: lidar fram fixed and added correctly

File: reccobot_description/urdf/camera.xacro (robot description, xacro)
@@ -3,6 +3,12 @@
     <gazebo reference="caml">
         <sensor name="camera" type="camera">
+            <pose> 0 0 0 0 0 0 </pose>
+            <visualize>true</visualize>
+            <always_on>true</always_on>
+            <update_rate>30</update_rate>
             <camera>
-                <horizontal_fov>1.0855</horizontal_fov> <image>
+                <camera_info_topic>camera/camera_info</camera_info_topic>
+                <horizontal_fov>1.0855</horizontal_fov>
+                <image>
                     <width>640</width>
                     <height>480</height>
@@ -19,17 +25,5 @@
                 </noise>
             </camera>
-            <always_on>1</always_on>
-            <update_rate>30</update_rate>
-            <visualize>true</visualize>
-            <plugin name="camera_controller" filename="libgz_ros_camera.so">
-                <ros>
-                    <namespace>/reccobot</namespace>
-                    <remapping>image_raw:=camera/image_raw</remapping>
-                    <remapping>camera_info:=camera/camera_info</remapping>
-                </ros>
-                <camera_name>camera</camera_name>
-                <frame_name>caml</frame_name>
-                <hack_baseline>0.07</hack_baseline>
-            </plugin>
+            <topic>camera/image_raw</topic>
         </sensor>
     </gazebo>

File: reccobot_description/urdf/lidar.xacro (robot description, xacro)
@@ -30,7 +30,8 @@
     <gazebo reference="lidarl">
         <material>Gazebo/Black</material>
-        <sensor name="laser" type="ray">
-            <pose> 0 0 0 0 0 0 </pose>
+        <sensor name="laser" type="gpu_ray">
+            <pose> -0.27 0.140 0.14345 -1.57 0 0.55 </pose>
             <visualize>true</visualize>
+            <always_on>true</always_on>
             <update_rate>10</update_rate>
             <ray>
@@ -54,11 +55,5 @@
                 </noise>
             </ray>
-            <plugin name="laser_controller" filename="libgz_ros_lidar_sensor.so">
-                <ros>
-                    <argument>~/out:=scan</argument>
-                </ros>
-                <output_type>sensor_msgs/LaserScan</output_type>
-                <frame_name>lidarl</frame_name>
-            </plugin>
+            <topic>scan</topic>
         </sensor>
     </gazebo>

File: reccobot_description/urdf/reccobot_core.xacro (robot description, xacro)
@@ -1,15 +1,6 @@
 <?xml version='1.0' encoding='utf-8'?>
-<robot name="reccobot_description" xmlns:xacro="http://www.ros.org/wiki/xacro">
-  <!-- Simulator selection forwarded from launch: Ignition/GZ vs Gazebo Classic -->
-  <xacro:arg name="is_ignition" default="true"/>
-  <!-- Sensor definitions and Gazebo plugins are embedded directly in this URDF -->
-  <!-- The xacro includes below are commented out to prevent xacro from ignoring the main robot body -->
-  <!--
-  <xacro:include filename="$(find reccobot_description)/urdf/lidar.xacro" />
-  <xacro:include filename="$(find reccobot_description)/urdf/camera.xacro" />
-  <xacro:include filename="$(find reccobot_description)/urdf/reccobot_ros2_control.xacro" />
-  <xacro:include filename="$(find reccobot_description)/urdf/reccobot_gazebo.xacro" />
-  -->
-  <!-- World link - fixed reference frame -->
+<robot xmlns:xacro="http://www.ros.org/wiki/xacro">
+  <!-- Base robot structure - links and joints only -->
+  <!-- Sensors and Gazebo plugins are in separate xacro files -->
   <!--
     ROTATION ADJUSTMENT:
@@ -1016,32 +1007,4 @@
     <axis xyz="0 0 0" />
   </joint>
-  <gazebo reference="caml">
-    <sensor name="camera" type="camera">
-      <pose> 0 0 0 0 0 0 </pose>
-      <visualize>true</visualize>
-      <always_on>true</always_on>
-      <update_rate>30</update_rate>
-      <camera>
-        <camera_info_topic>camera/camera_info</camera_info_topic>
-        <horizontal_fov>1.0855</horizontal_fov>
-        <image>
-          <width>640</width>
-          <height>480</height>
-          <format>R8G8B8</format>
-        </image>
-        <clip>
-          <near>0.1</near>
-          <far>100</far>
-        </clip>
-        <noise>
-          <type>gaussian</type>
-          <mean>0.0</mean>
-          <stddev>0.007</stddev>
-        </noise>
-      </camera>
-      <topic>camera/image_raw</topic>
-      <gz_frame_id>caml</gz_frame_id>
-    </sensor>
-  </gazebo>
   <link name="cell1">
     <inertial>
@@ -1299,63 +1262,5 @@
     <axis xyz="0 0 0" />
   </joint>
-  <link name="lidarl">
-    <inertial>
-      <origin xyz="-0.256143176414863 0.1283285607983 0.143452449615597" rpy="0 0 0" />
-      <mass value="0.109998846473485" />
-      <inertia ixx="4.02318810582621E-05" ixy="-7.76004870962997E-06" ixz="-7.75960890763623E-12" iyy="4.92541598732305E-05" iyz="-4.46080940664635E-12" izz="3.57666279058567E-05" />
-    </inertial>
-    <visual>
-      <origin xyz="0 0 0" rpy="0 0 0" />
-      <geometry>
-        <mesh filename="package://reccobot_description/meshes/lidarl.STL" />
-      </geometry>
-      <material name="">
-        <color rgba="0.659 0.333 0.969 1.0" />
-      </material>
-    </visual>
-    <collision>
-      <origin xyz="0 0 0" rpy="0 0 0" />
-      <geometry>
-        <mesh filename="package://reccobot_description/meshes/lidarl.STL" />
-      </geometry>
-    </collision>
-  </link>
-  <joint name="lidarmount_lidar" type="fixed">
-    <origin xyz="0 0 0" rpy="0 0 0" />
-    <parent link="lidarmount" />
-    <child link="lidarl" />
-    <axis xyz="0 0 0" />
-  </joint>
-  <gazebo reference="lidarl">
-    <material>Gazebo/Black</material>
-    <sensor name="laser" type="gpu_ray">
-      <pose> 0 0 0 0 0 0 </pose>
-      <visualize>true</visualize>
-      <always_on>true</always_on>
-      <update_rate>10</update_rate>
-      <ray>
-        <scan>
-          <horizontal>
-            <samples>500</samples>
-            <resolution>1</resolution>
-            <min_angle>-3.14159</min_angle>
-            <max_angle>3.14159</max_angle>
-          </horizontal>
-        </scan>
-        <range>
-          <min>0.05</min>
-          <max>12.0</max>
-          <resolution>0.015</resolution>
-        </range>
-        <noise>
-          <type>gaussian</type>
-          <mean>0.0</mean>
-          <stddev>0.01</stddev>
-        </noise>
-      </ray>
-      <topic>scan</topic>
-      <gz_frame_id>lidarl</gz_frame_id>
-    </sensor>
-  </gazebo>
+  <!-- lidarl link and joint are provided by lidar.xacro -->
   <link name="encoder">
     <inertial>

File: reccobot_description/urdf/reccobot_ros2_control.xacro (robot description, xacro)
@@ -5,8 +5,8 @@
   <xacro:property name="limit_servo" value="1.396" />
   <xacro:property name="limit_femur" value="${PI / 2}" />
-  <!-- ros2_control for Ignition Gazebo (ros_gz_sim) -->
+  <!-- ros2_control for Gazebo (ros_gz_sim) -->
   <ros2_control name="ReccobotSystem" type="system">
     <hardware>
-      <plugin>ign_ros2_control/IgnitionSystem</plugin>
+      <plugin>gz_ros2_control/GazeboSimSystem</plugin>
     </hardware>
     <!-- Legs: position-controlled servos (exclude passive feet joints) -->
@@ -119,7 +119,7 @@
     </joint>
   </ros2_control>
-  <!-- ros2_control plugin injection for Ignition Gazebo (ros_gz_sim) -->
+  <!-- ros2_control plugin injection for Gazebo (ros_gz_sim) -->
   <gazebo>
-    <plugin name="ign_ros2_control::IgnitionROS2ControlPlugin" filename="libign_ros2_control-system.so">
+    <plugin name="gz_ros2_control::GazeboSimROS2ControlPlugin" filename="libgz_ros2_control-system.so">
       <parameters>$(find reccobot_description)/config/reccobot_controllers.yaml</parameters>
     </plugin>

Commit message: all sensors working with correct frames and all

File: reccobot_description/urdf/camera.xacro (robot description, xacro)
@@ -1,5 +1,13 @@
 <?xml version="1.0"?>
 <robot xmlns:xacro="http://www.ros.org/wiki/xacro">
-    <gazebo reference="caml">
+    <link name="dummy_camera_link">
+    </link>
+    <joint name="caml_dummy_camera" type="fixed">
+        <!-- Position at actual sensor location, rotate 90° around Y (vertical scan) and 45° around Z (yaw) -->
+        <origin xyz="0 0 0" rpy="1.57 0 0" />
+        <parent link="caml" />
+        <child link="dummy_camera_link" />
+    </joint>
+    <gazebo reference="dummy_camera_link">
         <sensor name="camera" type="camera">
             <pose> 0 0 0 0 0 0 </pose>
@@ -25,4 +33,6 @@
                 </noise>
             </camera>
+            <gz_frame_id>dummy_camera_link</gz_frame_id>
+            <frame_name>dummy_camera_link</frame_name>
             <topic>camera/image_raw</topic>
         </sensor>

File: reccobot_description/urdf/lidar.xacro (robot description, xacro)
@@ -28,12 +28,22 @@
         <child link="lidarl" />
     </joint>
-    <gazebo reference="lidarl">
+    <!-- Add a rotated frame for the lidar sensor to publish vertical scans -->
+    <link name="lidarl_sensor">
+    </link>
+    <joint name="lidarl_lidarl_sensor" type="fixed">
+        <!-- Position at actual sensor location, rotate 90° around Y (vertical scan) and 45° around Z (yaw) -->
+        <origin xyz="-0.27 0.140 0.14345" rpy="0 1.5708 -1.05" />
+        <parent link="lidarl" />
+        <child link="lidarl_sensor" />
+    </joint>
+    <gazebo reference="lidarl_sensor">
         <material>Gazebo/Black</material>
-        <sensor name="laser" type="gpu_ray">
-            <pose> -0.27 0.140 0.14345 -1.57 0 0.55 </pose>
+        <sensor name="laser" type="gpu_lidar">
+            <!-- Sensor at origin of lidarl_sensor frame, no additional rotation -->
+            <pose>0 0 0 0 0 0</pose>
             <visualize>true</visualize>
             <always_on>true</always_on>
             <update_rate>10</update_rate>
-            <ray>
+            <lidar>
                 <scan>
                     <horizontal>
@@ -45,5 +55,5 @@
                 </scan>
                 <range>
-                    <min>0.05</min>
+                    <min>0.3</min>
                     <max>12.0</max>
                     <resolution>0.015</resolution>
@@ -54,5 +64,6 @@
                   <stddev>0.01</stddev>
                 </noise>
-            </ray>
+            </lidar>
+            <gz_frame_id>lidarl_sensor</gz_frame_id>
             <topic>scan</topic>
         </sensor>

File: reccobot_description/urdf/reccobot_description.urdf (robot description, URDF)
Before this commit: robot reccobot_description, 45 links, 44 joints
Links:
- link encoder: mass 0 -> 0.001

File: reccobot_description/urdf/reccobot_description.xacro (robot description, xacro)
@@ -14,3 +14,4 @@
     <xacro:include filename="lidar.xacro" />
     <xacro:include filename="camera.xacro" />
+    <xacro:include filename="imu.xacro" />
 </robot>

File: reccobot_description/urdf/reccobot_ros2_control.xacro (robot description, xacro)
@@ -118,4 +118,17 @@
       <state_interface name="position"/>
     </joint>
+    <!-- Passive feet joints - state-only (no command interface) -->
+    <joint name="feet1j">
+      <state_interface name="position"/>
+    </joint>
+    <joint name="feet2j">
+      <state_interface name="position"/>
+    </joint>
+    <joint name="feet3j">
+      <state_interface name="position"/>
+    </joint>
+    <joint name="feet4j">
+      <state_interface name="position"/>
+    </joint>
   </ros2_control>
   <!-- ros2_control plugin injection for Gazebo (ros_gz_sim) -->
