Commit message: lidar hardware plugin is working with step lag

File: reccobot_description/urdf/reccobot_core.xacro (robot description, xacro)
@@ -1202,5 +1202,5 @@
     <child link="coupling" />
     <axis xyz="1 0 0" />
-    <limit lower="-6.28" upper="6.25" effort="0.5" velocity="0.6" />
+    <limit lower="-6.28" upper="6.25" effort="5.0" velocity="6.0" />
     <dynamics damping="0.02" friction="0.01" />
     <safety_controller soft_upper_limit="6" soft_lower_limit="-6" k_position="5" k_velocity="0.2" />

File: reccobot_description/urdf/reccobot_description.urdf (robot description, URDF)
Before this commit: robot reccobot_description, 45 links, 44 joints
Joints:
- joint base_coupling: limit lower=-6.28 upper=6.25 effort=0.5 velocity=0.6 -> lower=-6.5 upper=6.5 effort=0.5 velocity=6.0

File: reccobot_description/urdf/reccobot_description.xacro (robot description, xacro)
@@ -2,5 +2,5 @@
 <robot xmlns:xacro="http://www.ros.org/wiki/xacro" name="reccobot">
     <xacro:arg name="use_ros2_control" default="true"/>
-    <xacro:arg name="sim_mode" default="false"/>
+    <xacro:arg name="sim_mode" default="true"/>
     <!-- Include the base robot structure -->
     <xacro:include filename="reccobot_core.xacro" />
@@ -9,6 +9,8 @@
         <xacro:include filename="reccobot_ros2_control.xacro" />
     </xacro:if>
-    <!-- Include Gazebo joint tuning -->
-    <xacro:include filename="reccobot_gazebo.xacro" />
+    <!-- Include Gazebo joint tuning (only for sim) -->
+    <xacro:if value="$(arg sim_mode)">
+        <xacro:include filename="reccobot_gazebo.xacro" />
+    </xacro:if>
     <!-- Include sensor definitions -->
     <xacro:include filename="lidar.xacro" />

File: reccobot_description/urdf/reccobot_gazebo.xacro (robot description, xacro)
@@ -158,10 +158,10 @@
 <!-- Lidar rotation joint (base_coupling) -->
 <gazebo reference="base_coupling">
-  <kp>5</kp>
-  <ki>0.0</ki>
-  <kd>0.5</kd>
+  <kp>100</kp>
+  <ki>0.5</ki>
+  <kd>5.0</kd>
   <friction>0.01</friction>
   <damping>0.02</damping>
-  <maxEffort>0.5</maxEffort>
+  <maxEffort>5.0</maxEffort>
   <provideFeedback>true</provideFeedback>
 </gazebo>

File: reccobot_description/urdf/reccobot_ros2_control.xacro (robot description, xacro)
@@ -1,140 +1,289 @@
 <?xml version="1.0"?>
 <robot xmlns:xacro="http://www.ros.org/wiki/xacro" name="reccobot">
-  <!-- Ignition/GZ plugin used unconditionally (launch uses ros_gz_sim) -->
+  <!-- Use sim_mode arg to switch between Gazebo sim and real hardware plugins -->
+  <xacro:arg name="sim_mode" default="true"/>
   <xacro:property name="PI" value="3.14159265359" />
   <xacro:property name="limit_servo" value="1.396" />
   <xacro:property name="limit_femur" value="${PI / 2}" />
-  <!-- ros2_control for Gazebo (ros_gz_sim) -->
-  <ros2_control name="ReccobotSystem" type="system">
-    <hardware>
-      <plugin>gz_ros2_control/GazeboSimSystem</plugin>
-    </hardware>
-    <!-- Legs: position-controlled servos (exclude passive feet joints) -->
-    <joint name="coxa1j">
-      <command_interface name="position">
-        <param name="min">${-limit_servo}</param>
-        <param name="max">${limit_servo}</param>
-      </command_interface>
-      <state_interface name="position"/>
-    </joint>
-    <joint name="femur1j">
-      <command_interface name="position">
-        <param name="min">${-limit_femur}</param>
-        <param name="max">${limit_femur}</param>
-      </command_interface>
-      <state_interface name="position"/>
-    </joint>
-    <joint name="tibia1j">
-      <command_interface name="position">
-        <param name="min">${-limit_servo}</param>
-        <param name="max">${limit_servo}</param>
-      </command_interface>
-      <state_interface name="position"/>
-    </joint>
-    <joint name="coxa2j">
-      <command_interface name="position">
-        <param name="min">${-limit_servo}</param>
-        <param name="max">${limit_servo}</param>
-      </command_interface>
-      <state_interface name="position"/>
-    </joint>
-    <joint name="femur2j">
-      <command_interface name="position">
-        <param name="min">${-limit_femur}</param>
-        <param name="max">${limit_femur}</param>
-      </command_interface>
-      <state_interface name="position"/>
-    </joint>
-    <joint name="tibia2j">
-      <command_interface name="position">
-        <param name="min">${-limit_servo}</param>
-        <param name="max">${limit_servo}</param>
-      </command_interface>
-      <state_interface name="position"/>
-    </joint>
-    <joint name="coxa3j">
-      <command_interface name="position">
-        <param name="min">${-limit_servo}</param>
-        <param name="max">${limit_servo}</param>
-      </command_interface>
-      <state_interface name="position"/>
-    </joint>
-    <joint name="femur3j">
-      <command_interface name="position">
-        <param name="min">${-limit_femur}</param>
-        <param name="max">${limit_femur}</param>
-      </command_interface>
-      <state_interface name="position"/>
-    </joint>
-    <joint name="tibia3j">
-      <command_interface name="position">
-        <param name="min">${-limit_servo}</param>
-        <param name="max">${limit_servo}</param>
-      </command_interface>
-      <state_interface name="position"/>
-    </joint>
-    <joint name="coxa4j">
-      <command_interface name="position">
-        <param name="min">${-limit_servo}</param>
-        <param name="max">${limit_servo}</param>
-      </command_interface>
-      <state_interface name="position"/>
-    </joint>
-    <joint name="femur4j">
-      <command_interface name="position">
-        <param name="min">${-limit_femur}</param>
-        <param name="max">${limit_femur}</param>
-      </command_interface>
-      <state_interface name="position"/>
-    </joint>
-    <joint name="tibia4j">
-      <command_interface name="position">
-        <param name="min">${-limit_servo}</param>
-        <param name="max">${limit_servo}</param>
-      </command_interface>
-      <state_interface name="position"/>
-    </joint>
-    <!-- Optional: camera gimbal joints -->
-    <joint name="cambase_caml1">
-      <command_interface name="position">
-        <param name="min">${-limit_servo}</param>
-        <param name="max">${limit_servo}</param>
-      </command_interface>
-      <state_interface name="position"/>
-    </joint>
-    <joint name="caml1_caml2">
-      <command_interface name="position">
-        <param name="min">${-limit_servo}</param>
-        <param name="max">${limit_servo}</param>
-      </command_interface>
-      <state_interface name="position"/>
-    </joint>
-    <!-- Lidar rotation joint -->
-    <joint name="base_coupling">
-      <command_interface name="position">
-        <param name="min">-6.28</param>
-        <param name="max">6.28</param>
-      </command_interface>
-      <state_interface name="position"/>
-    </joint>
-    <!-- Passive feet joints - state-only (no command interface) -->
-    <joint name="feet1j">
-      <state_interface name="position"/>
-    </joint>
-    <joint name="feet2j">
-      <state_interface name="position"/>
-    </joint>
-    <joint name="feet3j">
-      <state_interface name="position"/>
-    </joint>
-    <joint name="feet4j">
-      <state_interface name="position"/>
-    </joint>
-  </ros2_control>
-  <!-- ros2_control plugin injection for Gazebo (ros_gz_sim) -->
-  <gazebo>
-    <plugin name="gz_ros2_control::GazeboSimROS2ControlPlugin" filename="libgz_ros2_control-system.so">
-      <parameters>$(find reccobot_description)/config/reccobot_controllers.yaml</parameters>
-    </plugin>
-  </gazebo>
+  <!-- ==================== SIMULATION MODE ==================== -->
+  <xacro:if value="$(arg sim_mode)">
+    <!-- ros2_control for Gazebo (ros_gz_sim) - all joints use Gazebo plugin -->
+    <ros2_control name="ReccobotSystem" type="system">
+      <hardware>
+        <plugin>gz_ros2_control/GazeboSimSystem</plugin>
+      </hardware>
+      <!-- Legs: position-controlled servos (exclude passive feet joints) -->
+      <joint name="coxa1j">
+        <command_interface name="position">
+          <param name="min">${-limit_servo}</param>
+          <param name="max">${limit_servo}</param>
+        </command_interface>
+        <state_interface name="position"/>
+      </joint>
+      <joint name="femur1j">
+        <command_interface name="position">
+          <param name="min">${-limit_femur}</param>
+          <param name="max">${limit_femur}</param>
+        </command_interface>
+        <state_interface name="position"/>
+      </joint>
+      <joint name="tibia1j">
+        <command_interface name="position">
+          <param name="min">${-limit_servo}</param>
+          <param name="max">${limit_servo}</param>
+        </command_interface>
+        <state_interface name="position"/>
+      </joint>
+      <joint name="coxa2j">
+        <command_interface name="position">
+          <param name="min">${-limit_servo}</param>
+          <param name="max">${limit_servo}</param>
+        </command_interface>
+        <state_interface name="position"/>
+      </joint>
+      <joint name="femur2j">
+        <command_interface name="position">
+          <param name="min">${-limit_femur}</param>
+          <param name="max">${limit_femur}</param>
+        </command_interface>
+        <state_interface name="position"/>
+      </joint>
+      <joint name="tibia2j">
+        <command_interface name="position">
+          <param name="min">${-limit_servo}</param>
+          <param name="max">${limit_servo}</param>
+        </command_interface>
+        <state_interface name="position"/>
+      </joint>
+      <joint name="coxa3j">
+        <command_interface name="position">
+          <param name="min">${-limit_servo}</param>
+          <param name="max">${limit_servo}</param>
+        </command_interface>
+        <state_interface name="position"/>
+      </joint>
+      <joint name="femur3j">
+        <command_interface name="position">
+          <param name="min">${-limit_femur}</param>
+          <param name="max">${limit_femur}</param>
+        </command_interface>
+        <state_interface name="position"/>
+      </joint>
+      <joint name="tibia3j">
+        <command_interface name="position">
+          <param name="min">${-limit_servo}</param>
+          <param name="max">${limit_servo}</param>
+        </command_interface>
+        <state_interface name="position"/>
+      </joint>
+      <joint name="coxa4j">
+        <command_interface name="position">
+          <param name="min">${-limit_servo}</param>
+          <param name="max">${limit_servo}</param>
+        </command_interface>
+        <state_interface name="position"/>
+      </joint>
+      <joint name="femur4j">
+        <command_interface name="position">
+          <param name="min">${-limit_femur}</param>
+          <param name="max">${limit_femur}</param>
+        </command_interface>
+        <state_interface name="position"/>
+      </joint>
+      <joint name="tibia4j">
+        <command_interface name="position">
+          <param name="min">${-limit_servo}</param>
+          <param name="max">${limit_servo}</param>
+        </command_interface>
+        <state_interface name="position"/>
+      </joint>
+      <!-- Optional: camera gimbal joints -->
+      <joint name="cambase_caml1">
+        <command_interface name="position">
+          <param name="min">${-limit_servo}</param>
+          <param name="max">${limit_servo}</param>
+        </command_interface>
+        <state_interface name="position"/>
+      </joint>
+      <joint name="caml1_caml2">
+        <command_interface name="position">
+          <param name="min">${-limit_servo}</param>
+          <param name="max">${limit_servo}</param>
+        </command_interface>
+        <state_interface name="position"/>
+      </joint>
+      <!-- Lidar rotation joint -->
+      <joint name="base_coupling">
+        <command_interface name="position">
+          <param name="min">-6.28</param>
+          <param name="max">6.28</param>
+        </command_interface>
+        <state_interface name="position"/>
+        <state_interface name="velocity"/>
+        <state_interface name="effort"/>
+      </joint>
+      <!-- Passive feet joints - state-only (no command interface) -->
+      <joint name="feet1j">
+        <state_interface name="position"/>
+      </joint>
+      <joint name="feet2j">
+        <state_interface name="position"/>
+      </joint>
+      <joint name="feet3j">
+        <state_interface name="position"/>
+      </joint>
+      <joint name="feet4j">
+        <state_interface name="position"/>
+      </joint>
+    </ros2_control>
+    <!-- ros2_control plugin injection for Gazebo (ros_gz_sim) -->
+    <gazebo>
+      <plugin name="gz_ros2_control::GazeboSimROS2ControlPlugin" filename="libgz_ros2_control-system.so">
+        <parameters>$(find reccobot_description)/config/reccobot_controllers.yaml</parameters>
+      </plugin>
+    </gazebo>
+  </xacro:if>
+  <!-- ==================== REAL HARDWARE MODE ==================== -->
+  <xacro:unless value="$(arg sim_mode)">
+    <!-- ros2_control for real hardware legs + camera: use mock plugin for now -->
+    <ros2_control name="ReccobotLegsCameraSystem" type="system">
+      <hardware>
+        <!-- For now, use mock plugin; replace with your actual hardware plugin later -->
+        <plugin>mock_components/GenericSystem</plugin>
+        <param name="mock_sensor_commands">false</param>
+      </hardware>
+      <!-- Legs: position-controlled servos -->
+      <joint name="coxa1j">
+        <command_interface name="position">
+          <param name="min">${-limit_servo}</param>
+          <param name="max">${limit_servo}</param>
+        </command_interface>
+        <state_interface name="position"/>
+      </joint>
+      <joint name="femur1j">
+        <command_interface name="position">
+          <param name="min">${-limit_femur}</param>
+          <param name="max">${limit_femur}</param>
+        </command_interface>
+        <state_interface name="position"/>
+      </joint>
+      <joint name="tibia1j">
+        <command_interface name="position">
+          <param name="min">${-limit_servo}</param>
+          <param name="max">${limit_servo}</param>
+        </command_interface>
+        <state_interface name="position"/>
+      </joint>
+      <joint name="coxa2j">
+        <command_interface name="position">
+          <param name="min">${-limit_servo}</param>
+          <param name="max">${limit_servo}</param>
+        </command_interface>
+        <state_interface name="position"/>
+      </joint>
+      <joint name="femur2j">
+        <command_interface name="position">
+          <param name="min">${-limit_femur}</param>
+          <param name="max">${limit_femur}</param>
+        </command_interface>
+        <state_interface name="position"/>
+      </joint>
+      <joint name="tibia2j">
+        <command_interface name="position">
+          <param name="min">${-limit_servo}</param>
+          <param name="max">${limit_servo}</param>
+        </command_interface>
+        <state_interface name="position"/>
+      </joint>
+      <joint name="coxa3j">
+        <command_interface name="position">
+          <param name="min">${-limit_servo}</param>
+          <param name="max">${limit_servo}</param>
+        </command_interface>
+        <state_interface name="position"/>
+      </joint>
+      <joint name="femur3j">
+        <command_interface name="position">
+          <param name="min">${-limit_femur}</param>
+          <param name="max">${limit_femur}</param>
+        </command_interface>
+        <state_interface name="position"/>
+      </joint>
+      <joint name="tibia3j">
+        <command_interface name="position">
+          <param name="min">${-limit_servo}</param>
+          <param name="max">${limit_servo}</param>
+        </command_interface>
+        <state_interface name="position"/>
+      </joint>
+      <joint name="coxa4j">
+        <command_interface name="position">
+          <param name="min">${-limit_servo}</param>
+          <param name="max">${limit_servo}</param>
+        </command_interface>
+        <state_interface name="position"/>
+      </joint>
+      <joint name="femur4j">
+        <command_interface name="position">
+          <param name="min">${-limit_femur}</param>
+          <param name="max">${limit_femur}</param>
+        </command_interface>
+        <state_interface name="position"/>
+      </joint>
+      <joint name="tibia4j">
+        <command_interface name="position">
+          <param name="min">${-limit_servo}</param>
+          <param name="max">${limit_servo}</param>
+        </command_interface>
+        <state_interface name="position"/>
+      </joint>
+      <!-- Camera gimbal joints -->
+      <joint name="cambase_caml1">
+        <command_interface name="position">
+          <param name="min">${-limit_servo}</param>
+          <param name="max">${limit_servo}</param>
+        </command_interface>
+        <state_interface name="position"/>
+      </joint>
+      <joint name="caml1_caml2">
+        <command_interface name="position">
+          <param name="min">${-limit_servo}</param>
+          <param name="max">${limit_servo}</param>
+        </command_interface>
+        <state_interface name="position"/>
+      </joint>
+      <!-- Passive feet joints - state-only -->
+      <joint name="feet1j">
+        <state_interface name="position"/>
+      </joint>
+      <joint name="feet2j">
+        <state_interface name="position"/>
+      </joint>
+      <joint name="feet3j">
+        <state_interface name="position"/>
+      </joint>
+      <joint name="feet4j">
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